File: sk6805_clock_colon.sch (KiCad schematic (older format))
At the start: 10 parts

Commit message: Update usb position, byline
Parts:
- D49, D50, D51, D52, D53, D54, D55, D56: symbol LED:SK6805_1515 -> shadow_box_sk6805-rescue:SK6805_1515-LED
Changed lines of the file:
@@
 EESchema Schematic File Version 4
-LIBS:shadow_box_sk6805-cache
-EELAYER 29 0
+EELAYER 30 0
 EELAYER END
 $Descr A4 11693 8268
@@
 DOUT
 $Comp
-L LED:SK6805_1515 D49
+L shadow_box_sk6805-rescue:SK6805_1515-LED D49
 U 1 1 5E9308FE
 P 4200 1150
@@
 $EndComp
 $Comp
-L LED:SK6805_1515 D50
+L shadow_box_sk6805-rescue:SK6805_1515-LED D50
 U 1 1 5E933144
 P 5050 1150
@@
 $EndComp
 $Comp
-L LED:SK6805_1515 D52
+L shadow_box_sk6805-rescue:SK6805_1515-LED D52
 U 1 1 5E935D94
 P 5050 1950
@@
 $EndComp
 $Comp
-L LED:SK6805_1515 D51
+L shadow_box_sk6805-rescue:SK6805_1515-LED D51
 U 1 1 5E935D9A
 P 4200 1950
@@
 $EndComp
 $Comp
-L LED:SK6805_1515 D53
+L shadow_box_sk6805-rescue:SK6805_1515-LED D53
 U 1 1 5E93D656
 P 4200 3100
@@
 $EndComp
 $Comp
-L LED:SK6805_1515 D54
+L shadow_box_sk6805-rescue:SK6805_1515-LED D54
 U 1 1 5E93D65C
 P 5050 3100
@@
 $EndComp
 $Comp
-L LED:SK6805_1515 D56
+L shadow_box_sk6805-rescue:SK6805_1515-LED D56
 U 1 1 5E93D662
 P 5050 3900
@@
 $EndComp
 $Comp
-L LED:SK6805_1515 D55
+L shadow_box_sk6805-rescue:SK6805_1515-LED D55
 U 1 1 5E93D668
 P 4200 3900
